Commit message: Carpeta puzzlebot_rviz

File: slam_ws/src/puzzlebot_rviz/urdf/puzzlebot.urdf (robot description, URDF)
Before this commit: robot puzzlebot, 4 links, 3 joints
Links:
- added link camera_frame_optical
Joints:
- added joint base_link_to_camera_frame: type fixed, parent base_link, child camera_frame_optical, origin xyz=0.1 0 0.048 rpy=${-pi/2} 0 ${-pi/2}
